Commit message: Added imu.urdf.xacro and updated rgbd_camera.urdf.xacro and lidar.urdf.xacro

File: mobile_robot_description/urdf/mobile_robot.urdf.xacro (robot description, xacro)
@@ -5,7 +5,9 @@
   <xacro:include filename="$(find mobile_robot_description)/urdf/sensors/rgbd_camera.urdf.xacro"/>
   <xacro:include filename="$(find mobile_robot_description)/urdf/sensors/lidar.urdf.xacro"/>
+  <xacro:include filename="$(find mobile_robot_description)/urdf/sensors/imu.urdf.xacro"/>
   <!-- CALL THE MACRO -->
   <xacro:mobile_robot_base prefix=""/>
   <xacro:rgbd_camera prefix=""/>
   <xacro:lidar_link parent="base_link" xyz="0.0 0.0 0.055" rpy="0 0 0"/>
+  <xacro:imu_link parent="base_link" xyz="0.0 0.0 0.1" rpy="0 0 0"/>
 </robot>

File: mobile_robot_description/urdf/sensors/lidar.urdf.xacro (robot description, xacro)
@@ -20,4 +20,12 @@
             </geometry>
         </collision>
+        <inertial>
+            <mass value="${lidar_mass}"/>
+            <inertia ixx="${(1/12) * lidar_mass * (3 * lidar_radius * lidar_radius + lidar_length * lidar_length)}"
+                iyy="${(1/12) * lidar_mass * (3 * lidar_radius * lidar_radius + lidar_length * lidar_length)}"
+                izz="${(1/2) * lidar_mass * lidar_radius * lidar_radius}"
+                ixy="0" ixz="0" iyz="0"/>
+            <origin xyz="0 0 0" rpy="0 0 0"/>
+        </inertial>
     </link>
     <joint name="lidar_joint" type="fixed">
@@ -27,7 +35,9 @@
     </joint>
     <gazebo reference="lidar_link">
-        <sensor type="ray" name="lidar_sensor">
+        <sensor type="gpu_lidar" name="lidar_sensor">
             <always_on>1</always_on>
             <update_rate>10.0</update_rate>
+            <topic>/scan</topic>
+            <frame>lidar_link</frame>
             <ray>
                 <scan>

File: mobile_robot_description/urdf/sensors/rgbd_camera.urdf.xacro (robot description, xacro)
@@ -47,5 +47,5 @@
     </joint>
     <gazebo reference="${prefix}rgbd_camera_link">
-        <sensor type="depth" name="rgbd_camera">
+        <sensor type="rgbd_camera" name="rgbd_camera">
             <always_on>1</always_on>
             <update_rate>30.0</update_rate>
@@ -62,6 +62,6 @@
                 </clip>
             </camera>
-            <gz_frame_id>rgbd_optical_frame</gz_frame_id>
-            <topic>camera</topic>
+            <frame>rgbd_camera_link</frame>
+            <topic>/camera</topic>
             <visualize>true</visualize>
         </sensor>
