Commit message: Added load_ros2_controller.launch.py

File: mobile_robot_description/urdf/control/diff_drive_ros2_control.urdf.xacro (robot description, xacro)
@@ -8,5 +8,5 @@
                 </xacro:if>
             </hardware>
-            <joint name="${prefix}left_wheel_joint">
+            <joint name="base_left_wheel_joint">
                 <command_interface name="velocity">
                     <param name="min">-20.0</param>
@@ -16,5 +16,5 @@
                 <state_interface name="position"/>
             </joint>
-            <joint name="${prefix}right_wheel_joint">
+            <joint name="base_right_wheel_joint">
                 <command_interface name="velocity">
                     <param name="min">-20.0</param>
