Commit message: Modified ros_gz_bridge.yaml, load_ros2_controllers.launvh.py and other files

File: mobile_robot_description/urdf/control/gazebo_sim_ros2_control.urdf.xacro (robot description, xacro)
@@ -1,9 +1,9 @@
-<?xml version="1.0"?>
-<robot xmlns:xacro="http://www.ros.org/wiki/xacro">
-    <xacro:macro name="load_gazebo_ros2_control" params="robot_name use_gazebo">
+<?xml version="1.0" ?>
+<robot xmlns:xacro="http://wiki.ros.org/xacro">
+    <xacro:macro name="load_gazebo_sim_ros2_control_plugin" params="robot_name use_gazebo">
         <xacro:if value="${use_gazebo}">
             <gazebo>
-                <plugin name="gz_ros2_control::GazeboSimROS2ControlPlugin" filename="gz_ros2_control-system">
-                    <parameters>$(find mobile_robot_description)/urdf/diff_drive_controller.yaml</parameters>
+                <plugin filename="gz_ros2_control-system" name="gz_ros2_control::GazeboSimROS2ControlPlugin">
+                    <parameters>$(find mobile_robot_description)/config/${robot_name}/ros2_controllers.yaml</parameters>
                     <ros>
                         <remapping>/controller_manager/robot_description:=/robot_description</remapping>

File: mobile_robot_description/urdf/control/mobile_robot_ros2_control.urdf.xacro (robot description, xacro)
@@ -1,6 +1,6 @@
 <?xml version="1.0"?>
 <robot xmlns:xacro="http://www.ros.org/wiki/xacro">
-    <xacro:macro name="diff_drive_ros2_control" params="prefix use_gazebo">
-        <ros2_control name="DiffDriveSystem" type="system">
+    <xacro:macro name="mobile_robot_ros2_control" params="prefix use_gazebo">
+        <ros2_control name="RobotSystem" type="system">
             <hardware>
                 <xacro:if value="${use_gazebo}">

File: mobile_robot_description/urdf/robots/mobile_robot.urdf.xacro (robot description, xacro)
@@ -5,5 +5,5 @@
   <xacro:include filename="$(find mobile_robot_description)/urdf/sensors/lidar.urdf.xacro"/>
   <xacro:include filename="$(find mobile_robot_description)/urdf/sensors/imu.urdf.xacro"/>
-  <xacro:include filename="$(find mobile_robot_description)/urdf/control/diff_drive_ros2_control.urdf.xacro"/>
+  <xacro:include filename="$(find mobile_robot_description)/urdf/control/mobile_robot_ros2_control.urdf.xacro"/>
   <xacro:include filename="$(find mobile_robot_description)/urdf/control/gazebo_sim_ros2_control.urdf.xacro"/>
   <xacro:mobile_robot_base/>
@@ -11,5 +11,5 @@
   <xacro:lidar_link parent="base_link" xyz="0.0 0.0 ${base_height/2 + lidar_length/2}" rpy="0 0 0"/>
   <xacro:imu_link parent="base_link" xyz="${-(base_length/2)-(imu_length/2)} ${(rgbd_camera_width/2)+(imu_width/2)+(offset)} 0" rpy="0 0 0"/>
-  <xacro:diff_drive_ros2_control prefix="" use_gazebo="true"/>
-  <xacro:load_gazebo_ros2_control robot_name="mobile_robot" use_gazebo="true"/>
+  <xacro:mobile_robot_ros2_control prefix="" use_gazebo="true"/>
+  <xacro:load_gazebo_sim_ros2_control_plugin robot_name="mobile_robot" use_gazebo="true"/>
 </robot>

Commit message: Replaced robot_state_publisher.launch.py with a cleaner code and few modifications in other files

File: mobile_robot_description/urdf/control/gazebo_sim_ros2_control.urdf.xacro (robot description, xacro)
@@ -4,9 +4,6 @@
         <xacro:if value="${use_gazebo}">
             <gazebo>
-                <plugin filename="gz_ros2_control-system" name="gz_ros2_control::GazeboSimROS2ControlPlugin">
+                <plugin filename="libgz_ros2_control-system.so" name="gz_ros2_control::GazeboSimROS2ControlPlugin">
                     <parameters>$(find mobile_robot_description)/config/${robot_name}/ros2_controllers.yaml</parameters>
-                    <ros>
-                        <remapping>/controller_manager/robot_description:=/robot_description</remapping>
-                    </ros>
                 </plugin>
             </gazebo>

File: mobile_robot_description/urdf/control/mobile_robot_ros2_control.urdf.xacro (robot description, xacro)
@@ -1,10 +1,8 @@
 <?xml version="1.0"?>
 <robot xmlns:xacro="http://www.ros.org/wiki/xacro">
-    <xacro:macro name="mobile_robot_ros2_control" params="prefix use_gazebo">
-        <ros2_control name="DiffDriveSystem" type="system">
+    <xacro:macro name="mobile_robot_ros2_control" params="use_gazebo">
+        <ros2_control name="RobotSystem" type="system">
             <hardware>
-                <xacro:if value="${use_gazebo}">
-                    <plugin>gz_ros2_control/GazeboSystem</plugin>
-                </xacro:if>
+                    <plugin>gz_ros2_control/GazeboSimSystem</plugin>
             </hardware>
             <joint name="base_left_wheel_joint">
@@ -13,6 +11,6 @@
                     <param name="max">20.0</param>
                 </command_interface>
+                <state_interface name="position"/>
                 <state_interface name="velocity"/>
-                <state_interface name="position"/>
             </joint>
             <joint name="base_right_wheel_joint">
@@ -21,6 +19,6 @@
                     <param name="max">20.0</param>
                 </command_interface>
+                <state_interface name="position"/>
                 <state_interface name="velocity"/>
-                <state_interface name="position"/>
             </joint>
         </ros2_control>

File: mobile_robot_description/urdf/robots/mobile_robot.urdf.xacro (robot description, xacro)
@@ -1,5 +1,5 @@
 <?xml version="1.0"?>
 <robot name="mobile_robot" xmlns:xacro="http://www.ros.org/wiki/xacro">
-  <xacro:include filename="$(find mobile_robot_description)/urdf/base/mobile_robot_base.urdf.xacro"/>
+  <xacro:include filename="$(find mobile_robot_description)/urdf/mech/mobile_robot_base.urdf.xacro"/>
   <xacro:include filename="$(find mobile_robot_description)/urdf/sensors/rgbd_camera.urdf.xacro"/>
   <xacro:include filename="$(find mobile_robot_description)/urdf/sensors/lidar.urdf.xacro"/>
@@ -7,9 +7,11 @@
   <xacro:include filename="$(find mobile_robot_description)/urdf/control/mobile_robot_ros2_control.urdf.xacro"/>
   <xacro:include filename="$(find mobile_robot_description)/urdf/control/gazebo_sim_ros2_control.urdf.xacro"/>
+  <xacro:include filename="$(find mobile_robot_description)/urdf/control/velocity_control_plugin.urdf.xacro"/>
   <xacro:mobile_robot_base/>
   <xacro:rgbd_camera/>
   <xacro:lidar_link parent="base_link" xyz="0.0 0.0 ${base_height/2 + lidar_length/2}" rpy="0 0 0"/>
   <xacro:imu_link parent="base_link" xyz="${-(base_length/2)-(imu_length/2)} ${(rgbd_camera_width/2)+(imu_width/2)+(offset)} 0" rpy="0 0 0"/>
-  <xacro:mobile_robot_ros2_control prefix="" use_gazebo="true"/>
+  <xacro:mobile_robot_ros2_control use_gazebo="true"/>
   <xacro:load_gazebo_sim_ros2_control_plugin robot_name="mobile_robot" use_gazebo="true"/>
+  <xacro:load_velocity_control_plugin use_gazebo="true"/>
 </robot>
