Commit message: Replaced hardcoded inertias with xacro properties

File: mobile_robot_description/urdf/base/mobile_robot_base.urdf.xacro (robot description, xacro)
@@ -6,5 +6,5 @@
 <xacro:property name="cylindrical_wheel_radius" value="0.07" />
 <xacro:property name="cylindrical_wheel_length" value="0.02" />
-<xacro:property name="caster_radius" value="0.04" />
+<xacro:property name="caster_wheel_radius" value="0.04" />
 <xacro:property name="base_mass" value="5.0" />
 <xacro:property name="cylindrical_wheel_mass" value="0.5" />
@@ -12,5 +12,5 @@
 <xacro:macro name="mobile_robot_base" params="prefix">
     <material name="green">
-        <color rgba="0.0 0.8 0.0 1.0"/>
+        <color rgba="0 0.8 0 1"/>
     </material>
     <material name="grey">
@@ -23,5 +23,5 @@
                 <box size="${base_length} ${base_width} ${base_height}"/>
             </geometry>
-            <origin xyz="0.0 0.0 0.0" rpy="0.0 0.0 0.0"/>
+            <origin xyz="0 0 0" rpy="0 0 0"/>
             <material name="green"/>
         </visual>
@@ -30,10 +30,12 @@
                 <box size="${base_length} ${base_width} ${base_height}"/>
             </geometry>
-            <origin xyz="0.0 0.0 0.0" rpy="0.0 0.0 0.0"/>
+            <origin xyz="0 0 0" rpy="0 0 0"/>
         </collision>
         <inertial>
-            <mass value="5.0"/>
-            <inertia ixx="0.039" ixy="0.0" ixz="0.0" iyy="0.107" iyz="0.0" izz="0.122"/>
-            <origin xyz="0.0 0.0 0.0" rpy="0.0 0.0 0.0"/>
+            <mass value="${base_mass}"/>
+            <inertia ixx="${(1/12) * base_mass * (base_width * base_width + base_height * base_height)}" ixy="0" ixz="0"
+                iyy="${(1/12) * base_mass * (base_length * base_length + base_height * base_height)}" iyz="0"
+                izz="${(1/12) * base_mass * (base_length * base_length + base_width * base_width)}"/>
+            <origin xyz="0 0 0" rpy="0 0 0"/>
         </inertial>
     </link>
@@ -43,5 +45,5 @@
                 <cylinder radius="${cylindrical_wheel_radius}" length="${cylindrical_wheel_length}"/>
             </geometry>
-            <origin xyz="0.0 0.0 0.0" rpy="0.0 0.0 0.0"/>
+            <origin xyz="0 0 0" rpy="0 0 0"/>
             <material name="grey"/>
         </visual>
@@ -50,10 +52,13 @@
                 <cylinder radius="${cylindrical_wheel_radius}" length="${cylindrical_wheel_length}"/>
             </geometry>
-            <origin xyz="0.0 0.0 0.0" rpy="1.5708 0.0 0.0"/>
+            <origin xyz="0 0 0" rpy="1.5708 0 0"/>
         </collision>
         <inertial>
             <mass value="${cylindrical_wheel_mass}"/>
-            <inertia ixx="0.0007" ixy="0.0" ixz="0.0" iyy="0.0012" iyz="0.0" izz="0.0007"/>
-            <origin xyz="0.0 0.0 0.0" rpy="0.0 0.0 0.0"/>
+            <inertia ixx="${(1/12) * cylindrical_wheel_mass * (3 * cylindrical_wheel_radius * cylindrical_wheel_radius + cylindrical_wheel_length * cylindrical_wheel_length)}"
+                iyy="${(1/2) * cylindrical_wheel_mass * cylindrical_wheel_radius * cylindrical_wheel_radius}"
+                izz="${(1/12) * cylindrical_wheel_mass * (3 * cylindrical_wheel_radius * cylindrical_wheel_radius + cylindrical_wheel_length * cylindrical_wheel_length)}"
+                ixy="0" ixz="0" iyz="0"/>
+            <origin xyz="0 0 0" rpy="0 0 0"/>
         </inertial>
     </link>
@@ -63,5 +68,5 @@
                 <cylinder radius="${cylindrical_wheel_radius}" length="${cylindrical_wheel_length}"/>
             </geometry>
-            <origin xyz="0.0 0.0 0.0" rpy="0.0 0.0 0.0"/>
+            <origin xyz="0 0 0" rpy="0 0 0"/>
             <material name="grey"/>
         </visual>
@@ -70,10 +75,13 @@
                 <cylinder radius="${cylindrical_wheel_radius}" length="${cylindrical_wheel_length}"/>
             </geometry>
-            <origin xyz="0.0 0.0 0.0" rpy="1.5708 0.0 0.0"/>
+            <origin xyz="0 0 0" rpy="1.5708 0 0"/>
         </collision>
         <inertial>
             <mass value="${cylindrical_wheel_mass}"/>
-            <inertia ixx="0.0007" ixy="0.0" ixz="0.0" iyy="0.0012" iyz="0.0" izz="0.0007"/>
-            <origin xyz="0.0 0.0 0.0" rpy="0.0 0.0 0.0"/>
+            <inertia ixx="${(1/12) * cylindrical_wheel_mass * (3 * cylindrical_wheel_radius * cylindrical_wheel_radius + cylindrical_wheel_length * cylindrical_wheel_length)}"
+                iyy="${(1/2) * cylindrical_wheel_mass * cylindrical_wheel_radius * cylindrical_wheel_radius}"
+                izz="${(1/12) * cylindrical_wheel_mass * (3 * cylindrical_wheel_radius * cylindrical_wheel_radius + cylindrical_wheel_length * cylindrical_wheel_length)}"
+                ixy="0" ixz="0" iyz="0"/>
+            <origin xyz="0 0 0" rpy="0 0 0"/>
         </inertial>
     </link>
@@ -81,19 +89,22 @@
         <visual>
             <geometry>
-                <sphere radius="${caster_radius}"/>
+                <sphere radius="${caster_wheel_radius}"/>
             </geometry>
-            <origin xyz="0.0 0.0 0.0" rpy="0.0 0.0 0.0"/>
+            <origin xyz="0 0 0" rpy="0 0 0"/>
             <material name="grey"/>
         </visual>
         <collision>
             <geometry>
-                <sphere radius="${caster_radius}"/>
+                <sphere radius="${caster_wheel_radius}"/>
             </geometry>
-            <origin xyz="-0.15 0.0 -0.06" rpy="0.0 0.0 0.0"/>
+            <origin xyz="-0.15 0 -0.06" rpy="0 0 0"/>
         </collision>
         <inertial>
             <mass value="${caster_wheel_mass}"/>
-            <inertia ixx="0.0001" ixy="0.0" ixz="0.0" iyy="0.0001" iyz="0.0" izz="0.0001"/>
-            <origin xyz="0.0 0.0 0.0" rpy="0.0 0.0 0.0"/>
+            <inertia ixx="${(2/5) * caster_wheel_mass * caster_wheel_radius * caster_wheel_radius}"
+                iyy="${(2/5) * caster_wheel_mass * caster_wheel_radius * caster_wheel_radius}"
+                izz="${(2/5) * caster_wheel_mass * caster_wheel_radius * caster_wheel_radius}"
+                ixy="0" ixz="0" iyz="0"/>
+            <origin xyz="0 0 0" rpy="0 0 0"/>
         </inertial>
     </link>
@@ -101,17 +112,17 @@
         <parent link="${prefix}base_footprint"/>
         <child link="${prefix}base_link"/>
-        <origin xyz="0.0 0.0 0.1" rpy="0.0 0.0 0.0"/>
+        <origin xyz="0 0 0.1" rpy="0 0 0"/>
     </joint>
     <joint name="${prefix}base_right_wheel_joint" type="continuous">
         <parent link="${prefix}base_link"/>
         <child link="${prefix}right_wheel_link"/>
-        <axis xyz="0 0 1"/>
-        <origin xyz="0.1 0.16 -0.03" rpy="1.5708 0.0 0.0"/>
+        <axis xyz="0 1 0"/>
+        <origin xyz="0.1 0.16 -0.03" rpy="1.5708 0 0"/>
     </joint>
     <joint name="${prefix}base_left_wheel_joint" type="continuous">
         <parent link="${prefix}base_link"/>
         <child link="${prefix}left_wheel_link"/>
-        <axis xyz="0 0 1"/>
-        <origin xyz="0.1 -0.16 -0.03" rpy="1.5708 0.0 0.0"/>
+        <axis xyz="0 1 0"/>
+        <origin xyz="0.1 -0.16 -0.03" rpy="1.5708 0 0"/>
     </joint>
     <joint name="${prefix}base_caster_wheel_joint" type="fixed">
@@ -119,5 +130,5 @@
         <child link="${prefix}caster_wheel"/>
         <axis xyz="0 0 1"/>
-        <origin xyz="-0.15 0.0 -0.06" rpy="0.0 0.0 0.0"/>
+        <origin xyz="-0.15 0 -0.06" rpy="0 0 0"/>
     </joint>
 </xacro:macro>

Commit message: Created rgbd_camera.urdf.xacro

File: mobile_robot_description/urdf/base/mobile_robot_base.urdf.xacro (robot description, xacro)
@@ -34,7 +34,8 @@
         <inertial>
             <mass value="${base_mass}"/>
-            <inertia ixx="${(1/12) * base_mass * (base_width * base_width + base_height * base_height)}" ixy="0" ixz="0"
-                iyy="${(1/12) * base_mass * (base_length * base_length + base_height * base_height)}" iyz="0"
-                izz="${(1/12) * base_mass * (base_length * base_length + base_width * base_width)}"/>
+            <inertia ixx="${(1/12) * base_mass * (base_width * base_width + base_height * base_height)}"
+                iyy="${(1/12) * base_mass * (base_length * base_length + base_height * base_height)}"
+                izz="${(1/12) * base_mass * (base_length * base_length + base_width * base_width)}"
+                ixy="0" ixz="0" iyz="0"/>
             <origin xyz="0 0 0" rpy="0 0 0"/>
         </inertial>

File: mobile_robot_description/urdf/mobile_robot.urdf.xacro (robot description, xacro)
@@ -3,5 +3,7 @@
   <!-- Include your base file -->
   <xacro:include filename="$(find mobile_robot_description)/urdf/base/mobile_robot_base.urdf.xacro"/>
+  <xacro:include filename="$(find mobile_robot_description)/urdf/sensors/rgbd_camera.urdf.xacro"/>
   <!-- CALL THE MACRO -->
   <xacro:mobile_robot_base prefix=""/>
+  <xacro:rgbd_camera prefix=""/>
 </robot>

Commit message: Updated sensors

File: mobile_robot_description/urdf/base/mobile_robot_base.urdf.xacro (robot description, xacro)
@@ -53,5 +53,5 @@
                 <cylinder radius="${cylindrical_wheel_radius}" length="${cylindrical_wheel_length}"/>
             </geometry>
-            <origin xyz="0 0 0" rpy="1.5708 0 0"/>
+            <origin xyz="0 0 0" rpy="0 0 0"/>
         </collision>
         <inertial>
@@ -61,5 +61,5 @@
                 izz="${(1/12) * cylindrical_wheel_mass * (3 * cylindrical_wheel_radius * cylindrical_wheel_radius + cylindrical_wheel_length * cylindrical_wheel_length)}"
                 ixy="0" ixz="0" iyz="0"/>
-            <origin xyz="0 0 0" rpy="0 0 0"/>
+            <origin xyz="0 0 0" rpy="1.5708 0 0"/>
         </inertial>
     </link>
@@ -76,5 +76,5 @@
                 <cylinder radius="${cylindrical_wheel_radius}" length="${cylindrical_wheel_length}"/>
             </geometry>
-            <origin xyz="0 0 0" rpy="1.5708 0 0"/>
+            <origin xyz="0 0 0" rpy="0 0 0"/>
         </collision>
         <inertial>
@@ -84,5 +84,5 @@
                 izz="${(1/12) * cylindrical_wheel_mass * (3 * cylindrical_wheel_radius * cylindrical_wheel_radius + cylindrical_wheel_length * cylindrical_wheel_length)}"
                 ixy="0" ixz="0" iyz="0"/>
-            <origin xyz="0 0 0" rpy="0 0 0"/>
+            <origin xyz="0 0 0" rpy="1.5708 0 0"/>
         </inertial>
     </link>
@@ -99,5 +99,5 @@
                 <sphere radius="${caster_wheel_radius}"/>
             </geometry>
-            <origin xyz="-0.15 0 -0.06" rpy="0 0 0"/>
+            <origin xyz="0 0 0" rpy="0 0 0"/>
         </collision>
         <inertial>

File: mobile_robot_description/urdf/mobile_robot.urdf.xacro (robot description, xacro)
@@ -10,4 +10,4 @@
   <xacro:rgbd_camera prefix=""/>
   <xacro:lidar_link parent="base_link" xyz="0.0 0.0 0.055" rpy="0 0 0"/>
-  <xacro:imu_link parent="base_link" xyz="0.0 0.0 0.1" rpy="0 0 0"/>
+  <xacro:imu_link parent="base_link" xyz="0.2 0.0 0.05" rpy="0 0 0"/>
 </robot>

File: mobile_robot_description/urdf/sensors/imu.urdf.xacro (robot description, xacro)
@@ -1,11 +1,11 @@
 <?xml version="1.0"?>
 <robot xmlns:xacro="http://www.ros.org/wiki/xacro">
-<xacro:property name="imu_length" value="0.02" />
-<xacro:property name="imu_width" value="0.02" />
-<xacro:property name="imu_height" value="0.01" />
+<xacro:property name="imu_length" value="0.04" />
+<xacro:property name="imu_width" value="0.04" />
+<xacro:property name="imu_height" value="0.02" />
 <xacro:property name="imu_mass" value="0.1" />
 <xacro:macro name="imu_link" params="parent xyz rpy">
-    <material name="blue">
-        <color rgba="0 0 1 1"/>
+    <material name="red">
+        <color rgba="0.8 0 0 1"/>
     </material>
     <link name="imu_link">
@@ -14,5 +14,5 @@
                 <box size="${imu_length} ${imu_width} ${imu_height}"/>
             </geometry>
-            <material name="blue"/>
+            <material name="red"/>
         </visual>
         <collision>
@@ -21,4 +21,12 @@
             </geometry>
         </collision>
+        <inertial>
+            <mass value="${imu_mass}"/>
+            <inertia ixx="${(1/12) * imu_mass * (imu_width * imu_width + imu_height * imu_height)}"
+                iyy="${(1/12) * imu_mass * (imu_length * imu_length + imu_height * imu_height)}"
+                izz="${(1/12) * imu_mass * (imu_length * imu_length + imu_width * imu_width)}"
+                ixy="0" ixz="0" iyz="0"/>
+            <origin xyz="0 0 0" rpy="0 0 0"/>
+        </inertial>
     </link>
     <joint name="imu_joint" type="fixed">

Commit message: Modified sensors with xacro properties

File: mobile_robot_description/urdf/base/mobile_robot_base.urdf.xacro (robot description, xacro)
@@ -4,4 +4,5 @@
 <xacro:property name="base_width" value="0.3" />
 <xacro:property name="base_height" value="0.08" />
+<xacro:property name="offset" value="0.01" />
 <xacro:property name="cylindrical_wheel_radius" value="0.07" />
 <xacro:property name="cylindrical_wheel_length" value="0.02" />

File: mobile_robot_description/urdf/mobile_robot.urdf.xacro (robot description, xacro)
@@ -1,13 +1,11 @@
 <?xml version="1.0"?>
 <robot name="mobile_robot" xmlns:xacro="http://www.ros.org/wiki/xacro">
-  <!-- Include your base file -->
   <xacro:include filename="$(find mobile_robot_description)/urdf/base/mobile_robot_base.urdf.xacro"/>
   <xacro:include filename="$(find mobile_robot_description)/urdf/sensors/rgbd_camera.urdf.xacro"/>
   <xacro:include filename="$(find mobile_robot_description)/urdf/sensors/lidar.urdf.xacro"/>
   <xacro:include filename="$(find mobile_robot_description)/urdf/sensors/imu.urdf.xacro"/>
-  <!-- CALL THE MACRO -->
   <xacro:mobile_robot_base prefix=""/>
   <xacro:rgbd_camera prefix=""/>
-  <xacro:lidar_link parent="base_link" xyz="0.0 0.0 0.055" rpy="0 0 0"/>
-  <xacro:imu_link parent="base_link" xyz="0.2 0.0 0.05" rpy="0 0 0"/>
+  <xacro:lidar_link parent="base_link" xyz="0.0 0.0 ${base_height/2 + lidar_length/2}" rpy="0 0 0"/>
+  <xacro:imu_link parent="base_link" xyz="${-(base_length/2)-(imu_length/2)} ${(rgbd_camera_width/2)+(imu_width/2)+(offset)} 0" rpy="0 0 0"/>
 </robot>

File: mobile_robot_description/urdf/sensors/imu.urdf.xacro (robot description, xacro)
@@ -1,7 +1,7 @@
 <?xml version="1.0"?>
 <robot xmlns:xacro="http://www.ros.org/wiki/xacro">
-<xacro:property name="imu_length" value="0.04" />
+<xacro:property name="imu_length" value="0.02" />
 <xacro:property name="imu_width" value="0.04" />
-<xacro:property name="imu_height" value="0.02" />
+<xacro:property name="imu_height" value="0.04" />
 <xacro:property name="imu_mass" value="0.1" />
 <xacro:macro name="imu_link" params="parent xyz rpy">

Commit message: Modified robot_state_publisher.launch.py and other files

File: mobile_robot_description/urdf/base/mobile_robot_base.urdf.xacro (robot description, xacro)
@@ -11,5 +11,5 @@
 <xacro:property name="cylindrical_wheel_mass" value="0.5" />
 <xacro:property name="caster_wheel_mass" value="0.3" />
-<xacro:macro name="mobile_robot_base" params="prefix">
+<xacro:macro name="mobile_robot_base">
     <material name="green">
         <color rgba="0 0.8 0 1"/>
@@ -18,6 +18,6 @@
         <color rgba="0.8 0.8 0.8 1.0"/>
     </material>
-    <link name="${prefix}base_footprint" />
-    <link name="${prefix}base_link">
+    <link name="base_footprint" />
+    <link name="base_link">
         <visual>
             <geometry>
@@ -42,10 +42,10 @@
         </inertial>
     </link>
-    <link name="${prefix}right_wheel_link">
+    <link name="right_wheel_link">
         <visual>
             <geometry>
                 <cylinder radius="${cylindrical_wheel_radius}" length="${cylindrical_wheel_length}"/>
             </geometry>
-            <origin xyz="0 0 0" rpy="0 0 0"/>
+            <origin xyz="0 0 0" rpy="1.5708 0 0"/>
             <material name="grey"/>
         </visual>
@@ -54,5 +54,5 @@
                 <cylinder radius="${cylindrical_wheel_radius}" length="${cylindrical_wheel_length}"/>
             </geometry>
-            <origin xyz="0 0 0" rpy="0 0 0"/>
+            <origin xyz="0 0 0" rpy="1.5708 0 0"/>
         </collision>
         <inertial>
@@ -62,13 +62,13 @@
                 izz="${(1/12) * cylindrical_wheel_mass * (3 * cylindrical_wheel_radius * cylindrical_wheel_radius + cylindrical_wheel_length * cylindrical_wheel_length)}"
                 ixy="0" ixz="0" iyz="0"/>
-            <origin xyz="0 0 0" rpy="1.5708 0 0"/>
+            <origin xyz="0 0 0" rpy="0 0 0"/>
         </inertial>
     </link>
-    <link name="${prefix}left_wheel_link">
+    <link name="left_wheel_link">
         <visual>
             <geometry>
                 <cylinder radius="${cylindrical_wheel_radius}" length="${cylindrical_wheel_length}"/>
             </geometry>
-            <origin xyz="0 0 0" rpy="0 0 0"/>
+            <origin xyz="0 0 0" rpy="1.5708 0 0"/>
             <material name="grey"/>
         </visual>
@@ -77,5 +77,5 @@
                 <cylinder radius="${cylindrical_wheel_radius}" length="${cylindrical_wheel_length}"/>
             </geometry>
-            <origin xyz="0 0 0" rpy="0 0 0"/>
+            <origin xyz="0 0 0" rpy="1.5708 0 0"/>
         </collision>
         <inertial>
@@ -85,8 +85,8 @@
                 izz="${(1/12) * cylindrical_wheel_mass * (3 * cylindrical_wheel_radius * cylindrical_wheel_radius + cylindrical_wheel_length * cylindrical_wheel_length)}"
                 ixy="0" ixz="0" iyz="0"/>
-            <origin xyz="0 0 0" rpy="1.5708 0 0"/>
+            <origin xyz="0 0 0" rpy="0 0 0"/>
         </inertial>
     </link>
-    <link name="${prefix}caster_wheel">
+    <link name="caster_wheel">
         <visual>
             <geometry>
@@ -111,24 +111,24 @@
         </inertial>
     </link>
-    <joint name="${prefix}base_footprint_joint" type="fixed">
-        <parent link="${prefix}base_footprint"/>
-        <child link="${prefix}base_link"/>
+    <joint name="base_footprint_joint" type="fixed">
+        <parent link="base_footprint"/>
+        <child link="base_link"/>
         <origin xyz="0 0 0.1" rpy="0 0 0"/>
     </joint>
-    <joint name="${prefix}base_right_wheel_joint" type="continuous">
-        <parent link="${prefix}base_link"/>
-        <child link="${prefix}right_wheel_link"/>
+    <joint name="base_right_wheel_joint" type="continuous">
+        <parent link="base_link"/>
+        <child link="right_wheel_link"/>
         <axis xyz="0 1 0"/>
-        <origin xyz="0.1 0.16 -0.03" rpy="1.5708 0 0"/>
+        <origin xyz="0.1 0.16 -0.03" rpy="0 0 0"/>
     </joint>
-    <joint name="${prefix}base_left_wheel_joint" type="continuous">
-        <parent link="${prefix}base_link"/>
-        <child link="${prefix}left_wheel_link"/>
+    <joint name="base_left_wheel_joint" type="continuous">
+        <parent link="base_link"/>
+        <child link="left_wheel_link"/>
         <axis xyz="0 1 0"/>
-        <origin xyz="0.1 -0.16 -0.03" rpy="1.5708 0 0"/>
+        <origin xyz="0.1 -0.16 -0.03" rpy="0 0 0"/>
     </joint>
-    <joint name="${prefix}base_caster_wheel_joint" type="fixed">
-        <parent link="${prefix}base_link"/>
-        <child link="${prefix}caster_wheel"/>
+    <joint name="base_caster_wheel_joint" type="fixed">
+        <parent link="base_link"/>
+        <child link="caster_wheel"/>
         <axis xyz="0 0 1"/>
         <origin xyz="-0.15 0 -0.06" rpy="0 0 0"/>

File: mobile_robot_description/urdf/robots/mobile_robot.urdf.xacro (robot description, xacro)
@@ -7,6 +7,6 @@
   <xacro:include filename="$(find mobile_robot_description)/urdf/control/diff_drive_ros2_control.urdf.xacro"/>
   <xacro:include filename="$(find mobile_robot_description)/urdf/control/gazebo_sim_ros2_control.urdf.xacro"/>
-  <xacro:mobile_robot_base prefix=""/>
-  <xacro:rgbd_camera prefix=""/>
+  <xacro:mobile_robot_base/>
+  <xacro:rgbd_camera/>
   <xacro:lidar_link parent="base_link" xyz="0.0 0.0 ${base_height/2 + lidar_length/2}" rpy="0 0 0"/>
   <xacro:imu_link parent="base_link" xyz="${-(base_length/2)-(imu_length/2)} ${(rgbd_camera_width/2)+(imu_width/2)+(offset)} 0" rpy="0 0 0"/>

File: mobile_robot_description/urdf/sensors/rgbd_camera.urdf.xacro (robot description, xacro)
@@ -8,9 +8,9 @@
 <xacro:property name="base_width" value="0.3" />
 <xacro:property name="base_height" value="0.08" />
-<xacro:macro name="rgbd_camera" params="prefix">
+<xacro:macro name="rgbd_camera">
     <material name="blue">
         <color rgba="0 0 1 1"/>
     </material>
-    <link name="${prefix}rgbd_camera_link">
+    <link name="rgbd_camera_link">
         <visual>
             <geometry>
@@ -35,7 +35,7 @@
         </inertial>
     </link>
-    <joint name="${prefix}base_rgbd_camera_joint" type="fixed">
-        <parent link="${prefix}base_link"/>
-        <child link="${prefix}rgbd_camera_link"/>
+    <joint name="base_rgbd_camera_joint" type="fixed">
+        <parent link="base_link"/>
+        <child link="rgbd_camera_link"/>
         <origin xyz="${-(base_length/2)-(rgbd_camera_length/2)} 0 0" rpy="0 0 0"/>
     </joint>
@@ -46,5 +46,5 @@
       <origin xyz="0 0 0" rpy="-1.5708 0 -1.5708"/>
     </joint>
-    <gazebo reference="${prefix}rgbd_camera_link">
+    <gazebo reference="rgbd_camera_link">
         <sensor type="rgbd_camera" name="rgbd_camera">
             <always_on>1</always_on>
