Commit message: Completed Gazebo Simulation with keyboard teleop

File: mobile_description/urdf/mech/mobile_robot_base.urdf.xacro (robot description, xacro)
@@ -119,5 +119,5 @@
         <parent link="base_link"/>
         <child link="right_wheel_link"/>
-        <axis xyz="0 1 0"/>
+        <axis xyz="0 -1 0"/>
         <origin xyz="0.1 0.16 -0.03" rpy="0 0 0"/>
     </joint>
@@ -125,5 +125,5 @@
         <parent link="base_link"/>
         <child link="left_wheel_link"/>
-        <axis xyz="0 1 0"/>
+        <axis xyz="0 -1 0"/>
         <origin xyz="0.1 -0.16 -0.03" rpy="0 0 0"/>
     </joint>
@@ -148,4 +148,10 @@
         <fdir1>1 0 0</fdir1>
     </gazebo>
+    <gazebo reference="caster_wheel_link">
+        <mu1>0.001</mu1>
+        <mu2>0.001</mu2>
+        <kp>200000</kp>
+        <kd>2.0</kd>
+    </gazebo>
 </xacro:macro>
 </robot>

Commit message: Completed LiDAR scanning using cube, sphere, cone, etc.

File: mobile_description/urdf/mech/mobile_robot_base.urdf.xacro (robot description, xacro)
@@ -119,5 +119,5 @@
         <parent link="base_link"/>
         <child link="right_wheel_link"/>
-        <axis xyz="0 -1 0"/>
+        <axis xyz="0 1 0"/>
         <origin xyz="0.1 0.16 -0.03" rpy="0 0 0"/>
     </joint>
@@ -125,5 +125,5 @@
         <parent link="base_link"/>
         <child link="left_wheel_link"/>
-        <axis xyz="0 -1 0"/>
+        <axis xyz="0 1 0"/>
         <origin xyz="0.1 -0.16 -0.03" rpy="0 0 0"/>
     </joint>

File: mobile_description/urdf/robots/mobile_robot.urdf.xacro (robot description, xacro)
@@ -9,5 +9,5 @@
   <xacro:mobile_robot_base/>
   <xacro:rgbd_camera/>
-  <xacro:lidar_link parent="base_link" xyz="0.0 0.0 ${base_height/2 + lidar_length/2}" rpy="0 0 0"/>
+  <xacro:lidar_sensor parent="base_link" xyz="0.0 0.0 ${base_height/2 + lidar_length/2}" rpy="0 0 0"/>
   <xacro:imu_link parent="base_link" xyz="${-(base_length/2)-(imu_length/2)} ${(rgbd_camera_width/2)+(imu_width/2)+(offset)} 0" rpy="0 0 0"/>
   <xacro:mobile_robot_ros2_control use_gazebo="true"/>

File: mobile_description/urdf/sensors/lidar.urdf.xacro (robot description, xacro)
@@ -4,9 +4,9 @@
 <xacro:property name="lidar_length" value="0.03" />
 <xacro:property name="lidar_mass" value="0.2" />
-<xacro:macro name="lidar_link" params="parent xyz rpy">
+<xacro:macro name="lidar_sensor" params="parent xyz rpy">
     <material name="black">
         <color rgba="0 0 0 1"/>
     </material>
-    <link name="lidar_link">
+    <link name="laser_frame">
         <visual>
             <geometry>
@@ -29,15 +29,15 @@
         </inertial>
     </link>
-    <joint name="lidar_joint" type="fixed">
+    <joint name="laser_frame_joint" type="fixed">
         <parent link="${parent}"/>
-        <child link="lidar_link"/>
+        <child link="laser_frame"/>
         <origin xyz="${xyz}" rpy="${rpy}"/>
     </joint>
-    <gazebo reference="lidar_link">
+    <gazebo reference="laser_frame">
         <sensor type="gpu_lidar" name="lidar_sensor">
-            <always_on>1</always_on>
+            <always_on>true</always_on>
             <update_rate>10.0</update_rate>
-            <topic>/scan</topic>
-            <frame>lidar_link</frame>
+            <topic>scan</topic>
+            <visualize>false</visualize>
             <ray>
                 <scan>
@@ -48,11 +48,19 @@
                         <max_angle>3.14159</max_angle>
                     </horizontal>
+                    <vertical>
+                        <samples>1</samples>
+                        <resolution>1</resolution>
+                        <min_angle>0</min_angle>
+                        <max_angle>0</max_angle>
+                    </vertical>
                 </scan>
                 <range>
                     <min>0.1</min>
-                    <max>10.0</max>
+                    <max>30</max>
                     <resolution>0.01</resolution>
                 </range>
             </ray>
+            <gz_frame_id>laser_frame</gz_frame_id>
+            <frame_id>laser_frame</frame_id>
         </sensor>
     </gazebo>

Commit message: Modified nav2_default_view.rviz and mobile_robot_base.urdf.xacro

File: mobile_description/urdf/mech/mobile_robot_base.urdf.xacro (robot description, xacro)
@@ -119,5 +119,5 @@
         <parent link="base_link"/>
         <child link="right_wheel_link"/>
-        <axis xyz="0 1 0"/>
+        <axis xyz="0 -1 0"/>
         <origin xyz="0.1 0.16 -0.03" rpy="0 0 0"/>
     </joint>
@@ -125,5 +125,5 @@
         <parent link="base_link"/>
         <child link="left_wheel_link"/>
-        <axis xyz="0 1 0"/>
+        <axis xyz="0 -1 0"/>
         <origin xyz="0.1 -0.16 -0.03" rpy="0 0 0"/>
     </joint>

Commit message: Solved the issue where the robot doesn't rotates even when commands are given

File: mobile_description/urdf/mech/mobile_robot_base.urdf.xacro (robot description, xacro)
@@ -119,5 +119,5 @@
         <parent link="base_link"/>
         <child link="right_wheel_link"/>
-        <axis xyz="0 -1 0"/>
+        <axis xyz="0 1 0"/>
         <origin xyz="0.1 0.16 -0.03" rpy="0 0 0"/>
     </joint>
@@ -125,5 +125,5 @@
         <parent link="base_link"/>
         <child link="left_wheel_link"/>
-        <axis xyz="0 -1 0"/>
+        <axis xyz="0 1 0"/>
         <origin xyz="0.1 -0.16 -0.03" rpy="0 0 0"/>
     </joint>
@@ -139,5 +139,4 @@
         <kp>1000000.0</kp>
         <kd>10.0</kd>
-        <fdir1>1 0 0</fdir1>
     </gazebo>
     <gazebo reference="right_wheel_link">
@@ -146,11 +145,8 @@
         <kp>1000000.0</kp>
         <kd>10.0</kd>
-        <fdir1>1 0 0</fdir1>
     </gazebo>
     <gazebo reference="caster_wheel_link">
         <mu1>0.001</mu1>
         <mu2>0.001</mu2>
-        <kp>200000</kp>
-        <kd>2.0</kd>
     </gazebo>
 </xacro:macro>
